Commit message: Ya el continuous_lifter funciona en coopeliat

File: install/quadruped_model/share/quadruped_model/urdf/quadruped_SimpleModel.urdf (robot description, URDF)
Before this commit: robot quadruped_model, 9 links, 8 joints
Joints:
- removed joint foot_FRjoint
- added joint foot_FR_joint: type continuous, parent leg_FR_link, child foot_FR_link, origin xyz=-0.18217 -0.037449 0.00020128 rpy=0 0 0, axis 0 -1 0
